File: Hardware/Kicad/rf_attenuator_r3.kicad_sch (KiCad schematic)
At the start: 34 parts, among them J1 BNC, J2 BNC, SW1 SW_DPDT_x2, SW2 SW_DPDT_x2, SW3 SW_DPDT_x2, SW4 SW_DPDT_x2, SW5 SW_DPDT_x2, SW6 SW_DPDT_x2, SW7 SW_DPDT_x2

Commit message: Add files via upload
Parts:
- H1, H2, H3, H4: now left out of the parts list
- J1, J2: Vendor (none) -> Digikey; Vendor Part# (none) -> WM5514-ND
- R1: value 5.8 -> 5.9; Vendor (none) -> Digikey; Vendor Part# (none) -> 541-5.90AFCT-ND
- R10: value 37.3 -> 36; Vendor (none) -> Digikey; Vendor Part# (none) -> RMCF2512JT36ROCT-ND
- R11, R12: value 151 -> 150; Vendor (none) -> Digikey; Vendor Part# (none) -> 541-150AFCT-ND
- R13: value 71.2 -> 71.5; Vendor (none) -> Digikey; Vendor Part# (none) -> 541-71.5AFCT-ND
- R14, R15: value 96.2 -> 95.3; Vendor (none) -> Digikey; Vendor Part# (none) -> 541-95.3AFCT-ND
- R16, R19: value 242 -> 243; Vendor (none) -> Digikey; Vendor Part# (none) -> RMC2512FT243RCT-ND
- R17, R18, R20, R21: value 61.1 -> 61.9; Vendor (none) -> Digikey; Vendor Part# (none) -> 541-61.9AFCT-ND
- R2, R3: value 870 -> 866; Vendor (none) -> Digikey; Vendor Part# (none) -> 541-866AFCT-ND
- R4: value 11.6 -> 11.5; Vendor (none) -> Digikey; Vendor Part# (none) -> 541-11.5AFCT-ND
- R5, R6: value 436 -> 432; Vendor (none) -> Digikey; Vendor Part# (none) -> 119-CR2512-FX-4320ELFCT-ND
- R7: value 17.6 -> 17.8; Vendor (none) -> Digikey; Vendor Part# (none) -> 541-17.8AFCT-ND
- R8, R9: value 292 -> 294; Vendor (none) -> Digikey; Vendor Part# (none) -> 2019-RK73H3ATTE294OFCT-ND
- SW1, SW2, SW3, SW4, SW5, SW6, SW7: Vendor (none) -> Digikey; Vendor Part# (none) -> 401-2002-1-ND
